Commit message: get ik to be possible usable and limit thumb flexion of inspire hand

File: src/assets/inspire_hand/inspire_hand_right.urdf (robot description, URDF)
Before this commit: robot h1, 18 links, 17 joints
Joints:
- joint R_thumb_proximal_yaw_joint: limit lower=-0.1 upper=1.3 effort=1 velocity=0.5 -> lower=-0.1 upper=0.7 effort=1 velocity=0.5
