Commit message: update joint angles to new robot spec

File: src/assets/kbot/robot.urdf (robot description, URDF)
Before this commit: robot kbotv2p0_nohands, 13 links, 12 joints
Joints:
- joint dof_right_shoulder_pitch_03: limit lower=-3.141593 upper=1.396263 effort=60 velocity=18.849 -> lower=-3.49 upper=1.047 effort=60 velocity=18.849
- joint dof_right_shoulder_roll_03: limit lower=-1.658063 upper=0.349066 effort=60 velocity=18.849 -> lower=-1.658063 upper=0.436 effort=60 velocity=18.849

Commit message: fix left arm movement

File: src/assets/kbot/robot.urdf (robot description, URDF)
Before this commit: robot kbotv2p0_nohands, 13 links, 12 joints
Joints:
- joint dof_left_elbow_02: axis 0 0 -1 -> 0 0 1; origin xyz=-0.018500 0.010000 0.137000 rpy=-3.141593 1.570796 0 -> xyz=-0.018500 0.010000 0.137000 rpy=3.141593 1.570796 0
- joint dof_left_shoulder_pitch_03: limit lower=-1.396263 upper=3.141593 effort=60 velocity=18.849 -> lower=-1.047 upper=3.49 effort=60 velocity=18.849
- joint dof_left_shoulder_roll_03: limit lower=-0.349066 upper=1.658063 effort=60 velocity=18.849 -> lower=-0.436 upper=1.658063 effort=60 velocity=18.849

Commit message: fix left shoulder ROM

File: src/assets/kbot/robot.urdf (robot description, URDF)
Before this commit: robot kbotv2p0_nohands, 13 links, 12 joints
Joints:
- joint dof_left_shoulder_pitch_03: axis 0 0 1 -> 0 0 -1

Commit message: flip some left arm axes

File: src/assets/kbot/robot.urdf (robot description, URDF)
Before this commit: robot kbotv2p0_nohands, 13 links, 12 joints
Joints:
- joint dof_left_elbow_02: axis 0 0 1 -> 0 0 -1
- joint dof_left_shoulder_pitch_03: axis 0 0 -1 -> 0 0 1
