Commit message: enabled pausing of streaming robot commands

File: webxrtest/public/robot.urdf (robot description, URDF)
Before this commit: robot assy_forurdf_copy_1, 14 links, 13 joints
Joints:
- joint dof_left_wrist_00: origin xyz=0.017350 -0.103000 0.018000 rpy=1.570796 -1.570796 0 -> xyz=0.017350 -0.103000 0.018000 rpy=1.570796 3.141592 0
- joint dof_right_wrist_00: origin xyz=0.017350 0.103000 0.018000 rpy=-1.570796 1.570796 0 -> xyz=0.017350 0.103000 0.018000 rpy=-1.570796 0 0
